File: remote/remote.kicad_pcb (KiCad board)
At the start: 2 copper layers, 32.6 x 48.9 mm, 31 parts, among them J1 Conn_01x02, J2 Conn_01x04, Q1 Q_NPN_BEC, U1 IRM-H638T, U2 E103-W05, U3 HT66F2390, U4 AMS1117-3.3, Y1 11.0592M

Commit message: add code and finish inferred transmit and receive with NEC
Parts:
- added J3: Conn_01x04, Connector_PinHeader_2.54mm:PinHeader_1x04_P2.54mm_Vertical, F.Cu at (215.9, 98.4)
Connections:
- U3 pad 1: unconnected-(U3-Pad1) -> /SCL
- U3 pad 3: unconnected-(U3-Pad3) -> /SDA
- U3 pad 31: /LED1 -> unconnected-(U3-Pad31)
- U3 pad 32: /LED2 -> unconnected-(U3-Pad32)
- U3 pad 43: unconnected-(U3-Pad43) -> /LED1
- U3 pad 44: unconnected-(U3-Pad44) -> /LED2
Routing:
- net /SDA: track 0.00 -> 18.9 mm, vias 0 -> 1
- net /SCL: track 0.00 -> 18.7 mm, vias 0 -> 1
- net /LED2: track 5.89 -> 13.6 mm, vias 0 -> 2
- net /LED1: track 8.09 -> 15.5 mm, vias 0 -> 2
- net +3V3: track 135.5 -> 142.6 mm, vias 4 -> 5
- net Net-(C6-Pad2): track 15.3 -> 17.2 mm
- net GND: vias 23 -> 25
Other:
- board size 32.6 x 48.9 mm -> 34.8 x 48.9 mm
